Commit message: evetry5

File: install/wamv_gazebo/share/wamv_gazebo/urdf/wamv_gazebo.urdf.xacro (robot description, xacro)
@@ -3,6 +3,6 @@
 <robot xmlns:xacro="http://ros.org/wiki/xacro"
        name="WAM-V">
-  <xacro:arg name="locked" default="false" />
-  <xacro:arg name="thruster_config" default="H" />
+  <xacro:arg name="locked" default="true" />
+  <xacro:arg name="thruster_config" default="X" />
   <xacro:arg name="front_camera_enabled" default="true" />
   <xacro:arg name="chase_camera_enabled" default="false" />
@@ -73,4 +73,8 @@
   <!-- === Decide if we lock the robot to the world === -->
   <xacro:if value="$(arg locked)">
+    <gazebo reference="wamv">
+      <static>true</static>
+    </gazebo>
+    <!--
     <gazebo>
       <link name="wamv_external_link"/>
@@ -85,16 +89,11 @@
         </axis2>
       </joint>
-      <joint name="wamv_external_riser" type="prismatic">
+      <joint name="wamv_external_fix_joint" type="fixed">
         <parent>world</parent>
         <child>wamv_external_link</child>
-        <axis>
-          <limit>
-            <lower>-3</lower>
-            <upper>3</upper>
-          </limit>
-          <xyz>0 0 1</xyz>
-        </axis>
+        <origin xyz="0 0 0" rpy="0 0 0" />
       </joint>
     </gazebo>
+    -->
   </xacro:if>
   <!-- === Sensors === -->
